Commit message: 볼록 껍질 충돌 메쉬 + MuJoCo 변환 도구 추가
원본 URDF 가 참조하던 *_collision.STL 이 존재하지 않아 앞서 경계상자로
대체했는데, 형상이 너무 뭉개져 링크별 볼록 껍질로 다시 만든다.
ODE / PhysX / MuJoCo 모두 볼록 형상을 선호하므로 세 엔진 모두 이득이다.

tools/gen_collision_meshes.py
  visual STL -> convex hull. PhysX 의 볼록체 정점 256 상한을 고려해 200 으로
  제한하고, 초과분은 방향 샘플링으로 극점을 남기며 솎는다(부피 99% 이상 유지).
  결과: 275,574 -> 5,514 삼각형 (50배 감축), 전 링크 정점 200 이하.

tools/urdf_to_mjcf.py
  MuJoCo 는 URDF 를 읽지만 그대로는 시뮬이 안 된다 — base_link 가 월드에
  용접되어 자유 베이스가 없고(dof 20, 26 이어야 함), 액추에이터가 안 생기고,
  지면/조명이 없다. 이 셋을 채우고 메쉬 경로를 절대경로로 고정한다.

[자기충돌] 볼록 껍질은 오목한 부분을 메우므로 인접하지 않은 링크끼리 겹친다.
실측 결과 Knee_pitch <-> Ankle_roll 이 자세와 무관하게 상시 25.2 mm 침투,
base_link <-> Elbow_pitch 가 1.4~2.1 mm 침투한다. MuJoCo 는 부모-자식 쌍만
자동으로 거르므로 조부모-손자 쌍이 남는다.

Gazebo 는 self_collide=false 라 무해하지만 MuJoCo 는 허위 접촉력이 계속
걸려 같은 로봇이 두 엔진에서 다르게 움직인다. 정책 교차 검증에 치명적이라
contype/conaffinity 로 MuJoCo 쪽 자기충돌을 차단해 Gazebo 와 맞춘다.
(자기충돌 12 -> 0, 지면 접촉 8 유지)

검증
  Gazebo  base z = 0.43146, joint_states 999.6 Hz (실시간 배율 약 1.0)
  MuJoCo  base z = 0.4311, dof 26, actuator 20, 자기충돌 0

Co-Authored-By: Claude Opus 5 <noreply@anthropic.com>

File: src/kubot26_pkgs/urdf/kubot26_pkgs.urdf (robot description, URDF)
Before this commit: robot kubot26_pkgs, 23 links, 22 joints
Links:
- link Head_pitch: geometry collision mesh filename=package://kubot26_pkgs/meshes/collision/Head_pitch_collisio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; visual mesh filename=package://kubot26_pkgs/meshes/Head_pitch.STL
- link L_Ankle_pitch: geometry collision mesh filename=package://kubot26_pkgs/meshes/collision/L_Ankle_pitch_colli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; visual mesh filename=package://kubot26_pkgs/meshes/L_Ankle_pitch.STL
- link L_Ankle_roll: geometry collision mesh filename=package://kubot26_pkgs/meshes/collision/L_Ankle_roll_collis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; visual mesh filename=package://kubot26_pkgs/meshes/L_Ankle_roll.STL
- link L_Elbow_pitch: geometry collision mesh filename=package://kubot26_pkgs/meshes/collision/L_Elbow_pitch_colli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; visual mesh filename=package://kubot26_pkgs/meshes/L_Elbow_pitch.STL
- link L_Foot: geometry collision mesh filename=package://kubot26_pkgs/meshes/collision/L_Foot_collision.STL; visual mesh filename=package://kubot26_pkgs/meshes/L_Foot.STL
- link L_Hand_pitch: geometry collision mesh filename=package://kubot26_pkgs/meshes/collision/L_Hand_pitch_collis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; visual mesh filename=package://kubot26_pkgs/meshes/L_Hand_pitch.STL
- link L_Hip_pitch: geometry collision mesh filename=package://kubot26_pkgs/meshes/collision/L_Hip_pitch_collisi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; visual mesh filename=package://kubot26_pkgs/meshes/L_Hip_pitch.STL
- link L_Hip_roll: geometry collision mesh filename=package://kubot26_pkgs/meshes/collision/L_Hip_roll_collisio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; visual mesh filename=package://kubot26_pkgs/meshes/L_Hip_roll.STL
- link L_Hip_yaw: geometry collision mesh filename=package://kubot26_pkgs/meshes/collision/L_Hip_yaw_collision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; visual mesh filename=package://kubot26_pkgs/meshes/L_Hip_yaw.STL
- link L_Knee_pitch: geometry collision mesh filename=package://kubot26_pkgs/meshes/collision/L_Knee_pitch_collis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; visual mesh filename=package://kubot26_pkgs/meshes/L_Knee_pitch.STL
- link L_Shoulder_roll: geometry collision mesh filename=package://kubot26_pkgs/meshes/collision/L_Shoulder_roll_col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; visual mesh filename=package://kubot26_pkgs/meshes/L_Shoulder_roll.STL
- link Neck_yaw: geometry collision mesh filename=package://kubot26_pkgs/meshes/collision/Neck_yaw_collision.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; visual mesh filename=package://kubot26_pkgs/meshes/Neck_yaw.STL
- link R_Ankle_pitch: geometry collision mesh filename=package://kubot26_pkgs/meshes/collision/R_Ankle_pitch_colli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; visual mesh filename=package://kubot26_pkgs/meshes/R_Ankle_pitch.STL
- link R_Ankle_roll: geometry collision mesh filename=package://kubot26_pkgs/meshes/collision/R_Ankle_roll_collis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; visual mesh filename=package://kubot26_pkgs/meshes/R_Ankle_roll.STL
- link R_Elbow_pitch: geometry collision mesh filename=package://kubot26_pkgs/meshes/collision/R_Elbow_pitch_colli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; visual mesh filename=package://kubot26_pkgs/meshes/R_Elbow_pitch.STL
- link R_Foot: geometry collision mesh filename=package://kubot26_pkgs/meshes/collision/R_Foot_collision.STL; visual mesh filename=package://kubot26_pkgs/meshes/R_Foot.STL
- link R_Hand_pitch: geometry collision mesh filename=package://kubot26_pkgs/meshes/collision/R_Hand_pitch_collis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; visual mesh filename=package://kubot26_pkgs/meshes/R_Hand_pitch.STL
- link R_Hip_pitch: geometry collision mesh filename=package://kubot26_pkgs/meshes/collision/R_Hip_pitch_collisi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; visual mesh filename=package://kubot26_pkgs/meshes/R_Hip_pitch.STL
- link R_Hip_roll: geometry collision mesh filename=package://kubot26_pkgs/meshes/collision/R_Hip_roll_collisio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; visual mesh filename=package://kubot26_pkgs/meshes/R_Hip_roll.STL
- link R_Hip_yaw: geometry collision mesh filename=package://kubot26_pkgs/meshes/collision/R_Hip_yaw_collision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; visual mesh filename=package://kubot26_pkgs/meshes/R_Hip_yaw.STL
- link R_Knee_pitch: geometry collision mesh filename=package://kubot26_pkgs/meshes/collision/R_Knee_pitch_collis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; visual mesh filename=package://kubot26_pkgs/meshes/R_Knee_pitch.STL
- link R_Shoulder_roll: geometry collision mesh filename=package://kubot26_pkgs/meshes/collision/R_Shoulder_roll_col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; visual mesh filename=package://kubot26_pkgs/meshes/R_Shoulder_roll.STL
- link base_link: geometry collision mesh filename=package://kubot26_pkgs/meshes/collision/base_link_collision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; visual mesh filename=package://kubot26_pkgs/meshes/base_link.STL
